Commit message: test end-to-end, test if torque control work or not

File: alpha_description/urdf/alpha_robot_for_pybullet.urdf (robot description, URDF)
Before this commit: robot alpha_robot, 13 links, 12 joints
Joints:
- joint joint_1: limit lower=0.032 upper=6.02 effort=54.36 velocity=100000 -> lower=0.032 upper=6.02 effort=54.36 velocity=10
- joint joint_2: limit lower=0.0174533 upper=3.40339 effort=54.36 velocity=100000 -> lower=0.0174533 upper=3.40339 effort=54.36 velocity=10
- joint joint_3: limit lower=0.0174533 upper=3.40339 effort=47.112 velocity=100000 -> lower=0.0174533 upper=3.40339 effort=47.112 velocity=10
- joint joint_4: limit lower=0.0 upper=3.22 effort=33.069 velocity=100000 -> lower=0.0 upper=3.22 effort=33.069 velocity=10
- joint joint_5: limit lower=0.0013 upper=0.0133 effort=28.992 velocity=100000 -> lower=0.0013 upper=0.0133 effort=28.992 velocity=10

Commit message: correct urdf file

File: alpha_description/urdf/alpha_robot_for_pybullet.urdf (robot description, URDF)
Before this commit: robot alpha_robot, 13 links, 12 joints
Links:
- removed link alpha_base_link
- removed link alpha_ee_base_link
- removed link alpha_m1_link
- removed link alpha_m2_1_1_link
- removed link alpha_m2_1_2_link
- removed link alpha_m2_joint_link
- removed link alpha_m3_inline_link
- removed link alpha_push_rod
- removed link alpha_standard_jaws_base_link
- removed link alpha_standard_jaws_rs1_130_link
- removed link alpha_standard_jaws_rs1_139_link
- removed link alpha_tcp
- added link base_link, mass 0.1; collision cylinder length=0.150 radius=0.020; visual mesh filename=meshes/RS1-1010.dae
- added link ee_base_link, mass 0.05
- added link m1_link, mass 0.200; collision cylinder length=0.1 radius=0.020; visual mesh filename=meshes/M1.dae
- added link m2_1_1_link, mass 0.194; collision cylinder length=0.033 radius=0.020; visual mesh filename=meshes/M2-1-1.dae
- added link m2_1_3_link, mass 0.115; collision cylinder length=0.033 radius=0.020; visual mesh filename=meshes/M2-1-3.dae
- added link m2_link, mass 0.429; collision cylinder length=0.040 radius=0.020; collision cylinder length=0.040 radius=0.020
- added link m3_inline_link, mass 0.341; collision cylinder length=0.150 radius=0.020; visual mesh filename=meshes/M3-INLINE.dae
- added link push_rod, mass 0.02
- added link standard_jaws_base_link, mass 0.03; visual mesh filename=meshes/end_effectors/RS1-124.stl
- added link standard_jaws_rs1_130_link, mass 0.02; collision box size=0.012 0.03 0.09; visual mesh filename=meshes/end_effectors/RS1-130.dae
- added link standard_jaws_rs1_139_link, mass 0.02; collision box size=0.012 0.03 0.09; visual mesh filename=meshes//end_effectors/RS1-139.dae
- added link tcp, mass 0.001
Joints:
- removed joint alpha_base_joint
- removed joint alpha_base_link_joint
- removed joint alpha_ee_joint
- removed joint alpha_standard_jaws_base_joint
- removed joint alpha_standard_jaws_rs1_130_joint
- removed joint alpha_standard_jaws_rs1_139_joint
- removed joint alpha_tcp_joint
- added joint base_joint: type fixed, parent world, child base_link, origin xyz=0 0 0 rpy=0 0 0
- added joint ee_joint: type fixed, parent m1_link, child ee_base_link, origin xyz=0 0 0.09975 rpy=0 0 0
- added joint mount_joint: type fixed, parent base_link, child m3_inline_link, origin xyz=0.124 0.004 0 rpy=0 0 0
- added joint standard_jaws_base_joint: type fixed, parent ee_base_link, child standard_jaws_base_link, origin xyz=0 0 0 rpy=0 0 0
- added joint standard_jaws_rs1_130_joint: type revolute, parent standard_jaws_base_link, child standard_jaws_rs1_130_link, origin xyz=0 0.0155 0.0069 rpy=0 0 0, axis -1 0 0, limit lower=0 upper=0.5 effort=10 velocity=10, mimic joint=joint_5 multiplier=41.67 offset=0
- added joint standard_jaws_rs1_139_joint: type revolute, parent standard_jaws_base_link, child standard_jaws_rs1_139_link, origin xyz=0 -0.0155 0.0069 rpy=0 0 0, axis 1 0 0, limit lower=0 upper=0.5 effort=10 velocity=10, mimic joint=standard_jaws_rs1_130_joint multiplier=1 offset=0
- added joint tcp_joint: type fixed, parent standard_jaws_base_link, child tcp, origin xyz=0 0 0.09 rpy=0 0 0
- joint joint_1: child alpha_m2_1_1_link -> m2_1_1_link; limit lower=0.032 upper=6.02 effort=54.36 velocity=10 -> lower=-3.072 upper=3.072 effort=9.0 velocity=0.5; origin xyz=0 0 0.014 rpy=0 0 0 -> xyz=0 0 0.014; parent alpha_m3_inline_link -> m3_inline_link
- joint joint_2: child alpha_m2_joint_link -> m2_link; limit lower=0.0174533 upper=3.40339 effort=54.36 velocity=10 -> lower=-1.745 upper=1.745 effort=9.0 velocity=0.5; origin xyz=-0.02 0 0.033 rpy=0 0 0 -> xyz=-0.02 0 0.033 rpy=0 1.745 0; parent alpha_m2_1_1_link -> m2_1_1_link
- joint joint_3: child alpha_m2_1_2_link -> m2_1_3_link; limit lower=0.0174533 upper=3.40339 effort=47.112 velocity=10 -> lower=-1.614 upper=1.614 effort=9.0 velocity=0.5; origin xyz=-0.04 0 -0.1453 rpy=0 0 0 -> xyz=-0.04 0 -0.1453 rpy=0 0.204 3.14159; parent alpha_m2_joint_link -> m2_link
- joint joint_4: child alpha_m1_link -> m1_link; limit lower=0.0 upper=3.22 effort=33.069 velocity=10 -> lower=-0.785 upper=0.785 effort=9.0 velocity=0.5; origin xyz=0.02 0 0.033 rpy=0 0 0 -> xyz=0.02 0 0.033 rpy=0 0 2.09439; parent alpha_m2_1_2_link -> m2_1_3_link
- joint joint_5: child alpha_push_rod -> push_rod; limit lower=0.0013 upper=0.0133 effort=28.992 velocity=10 -> lower=0.001 upper=0.013 effort=10 velocity=10; parent alpha_ee_base_link -> ee_base_link

File: alpha_description/urdf/alpha_robot_for_pybullet_test.urdf (robot description, URDF)
Before this commit: robot alpha_robot, 13 links, 12 joints
Links:
- removed link alpha_base_link
- removed link alpha_ee_base_link
- removed link alpha_m1_link
- removed link alpha_m2_1_1_link
- removed link alpha_m2_1_2_link
- removed link alpha_m2_joint_link
- removed link alpha_m3_inline_link
- removed link alpha_push_rod
- removed link alpha_standard_jaws_base_link
- removed link alpha_standard_jaws_rs1_130_link
- removed link alpha_standard_jaws_rs1_139_link
- removed link alpha_tcp
- added link base_link, mass 0.1; collision cylinder length=0.150 radius=0.020; visual mesh filename=meshes/RS1-1010.dae
- added link m1_link, mass 0.200; collision cylinder length=0.1 radius=0.020; visual mesh filename=meshes/M1.dae
- added link m2_1_1_link, mass 0.194; collision cylinder length=0.033 radius=0.020; visual mesh filename=meshes/M2-1-1.dae
- added link m2_1_3_link, mass 0.115; collision cylinder length=0.033 radius=0.020; visual mesh filename=meshes/M2-1-3.dae
- added link m2_link, mass 0.429; collision cylinder length=0.040 radius=0.020; collision cylinder length=0.040 radius=0.020
- added link m3_inline_link, mass 0.341; collision cylinder length=0.150 radius=0.020; visual mesh filename=meshes/M3-INLINE.dae
- added link push_rod, mass 0.001; visual box size=0.001 0.001 0.001
- added link rs1_124_link, mass 0.05; collision cylinder length=0.1 radius=0.020; visual mesh filename=meshes/RS1-124.dae
Joints:
- removed joint alpha_base_joint
- removed joint alpha_base_link_joint
- removed joint alpha_ee_joint
- removed joint alpha_standard_jaws_base_joint
- removed joint alpha_standard_jaws_rs1_130_joint
- removed joint alpha_standard_jaws_rs1_139_joint
- removed joint alpha_tcp_joint
- added joint base_joint: type fixed, parent world, child base_link, origin xyz=0 0 0 rpy=0 0 0
- added joint mount_joint: type fixed, parent base_link, child m3_inline_link, origin xyz=0.124 0.004 0 rpy=0 0 0
- added joint tcp_base_joint: type fixed, parent m1_link, child rs1_124_link, origin xyz=0 0 0.09975 rpy=0 0 0
- joint joint_1: child alpha_m2_1_1_link -> m2_1_1_link; limit lower=0.032 upper=6.02 effort=54.36 velocity=100000 -> lower=-3.072 upper=3.072 effort=9.0 velocity=0.5; origin xyz=0 0 0.014 rpy=0 0 0 -> xyz=0 0 0.014; parent alpha_m3_inline_link -> m3_inline_link
- joint joint_2: child alpha_m2_joint_link -> m2_link; limit lower=0.0174533 upper=3.40339 effort=54.36 velocity=100000 -> lower=-1.745 upper=1.745 effort=9.0 velocity=0.5; origin xyz=-0.02 0 0.033 rpy=0 0 0 -> xyz=-0.02 0 0.033 rpy=0 1.745 0; parent alpha_m2_1_1_link -> m2_1_1_link
- joint joint_3: child alpha_m2_1_2_link -> m2_1_3_link; limit lower=0.0174533 upper=3.40339 effort=47.112 velocity=100000 -> lower=-1.614 upper=1.614 effort=9.0 velocity=0.5; origin xyz=-0.04 0 -0.1453 rpy=0 0 0 -> xyz=-0.04 0 -0.1453 rpy=0 0.204 3.14159; parent alpha_m2_joint_link -> m2_link
- joint joint_4: child alpha_m1_link -> m1_link; limit lower=0.0 upper=3.22 effort=33.069 velocity=100000 -> lower=-0.785 upper=0.785 effort=9.0 velocity=0.5; origin xyz=0.02 0 0.033 rpy=0 0 0 -> xyz=0.02 0 0.033 rpy=0 0 2.09439; parent alpha_m2_1_2_link -> m2_1_3_link
- joint joint_5: child alpha_push_rod -> push_rod; limit lower=0.0013 upper=0.0133 effort=28.992 velocity=100000 -> lower=0.001 upper=0.013 effort=10 velocity=10; parent alpha_ee_base_link -> rs1_124_link

Commit message: big change and some result, trying to connect to real robot.

File: alpha_description/urdf/alpha_robot_for_pybullet.urdf (robot description, URDF)
Before this commit: robot alpha_robot, 13 links, 12 joints
Links:
- link base_link: geometry collision cylinder length=0.150 radius=0.03; visual mesh filename=meshes/RS1-1010.dae
- link m1_link: geometry collision cylinder length=0.1 radius=0.03; visual mesh filename=meshes/M1.dae
- link m2_1_1_link: geometry collision cylinder length=0.033 radius=0.03; visual mesh filename=meshes/M2-1-1.dae
- link m2_1_3_link: geometry collision cylinder length=0.033 radius=0.03; visual mesh filename=meshes/M2-1-3.dae
- link m2_link: geometry collision cylinder length=0.040 radius=0.03; collision cylinder length=0.040 radius=0.03
- link m3_inline_link: geometry collision cylinder length=0.150 radius=0.03; visual mesh filename=meshes/M3-INLINE.dae
Joints:
- joint joint_3: limit lower=-1.614 upper=1.614 effort=9.0 velocity=0.5 -> lower=-0.262 upper=2.094 effort=9.0 velocity=0.5
- joint joint_4: limit lower=-0.785 upper=0.785 effort=9.0 velocity=0.5 -> lower=-2.862 upper=2.862 effort=9.0 velocity=0.5

File: alpha_description/urdf/alpha_robot_for_pybullet_test.urdf (robot description, URDF)
Before this commit: robot alpha_robot, 9 links, 8 joints
Links:
- removed link rs1_124_link
- added link ee_base_link, mass 0.05
- added link standard_jaws_base_link, mass 0.03; visual mesh filename=meshes/end_effectors/RS1-124.stl
- added link standard_jaws_rs1_130_link, mass 0.02; collision box size=0.012 0.03 0.09; visual mesh filename=meshes/end_effectors/RS1-130.dae
- added link standard_jaws_rs1_139_link, mass 0.02; collision box size=0.012 0.03 0.09; visual mesh filename=meshes//end_effectors/RS1-139.dae
- added link tcp, mass 0.001
- link base_link: geometry collision cylinder length=0.150 radius=0.03; visual mesh filename=meshes/RS1-1010.dae
- link m1_link: geometry collision cylinder length=0.1 radius=0.03; visual mesh filename=meshes/M1.dae
- link m2_1_1_link: geometry collision cylinder length=0.033 radius=0.03; visual mesh filename=meshes/M2-1-1.dae
- link m2_1_3_link: geometry collision cylinder length=0.033 radius=0.03; visual mesh filename=meshes/M2-1-3.dae
- link m2_link: geometry collision cylinder length=0.040 radius=0.03; collision cylinder length=0.040 radius=0.03
- link m3_inline_link: geometry collision cylinder length=0.150 radius=0.03; visual mesh filename=meshes/M3-INLINE.dae
- link push_rod: mass 0.001 -> 0.02; geometry 
Joints:
- removed joint tcp_base_joint
- added joint ee_joint: type fixed, parent m1_link, child ee_base_link, origin xyz=0 0 0.09975 rpy=0 0 0
- added joint standard_jaws_base_joint: type fixed, parent ee_base_link, child standard_jaws_base_link, origin xyz=0 0 0 rpy=0 0 0
- added joint standard_jaws_rs1_130_joint: type revolute, parent standard_jaws_base_link, child standard_jaws_rs1_130_link, origin xyz=0 0.0155 0.0069 rpy=0 0 0, axis -1 0 0, limit lower=0 upper=0.5 effort=10 velocity=10, mimic joint=joint_5 multiplier=41.67 offset=0
- added joint standard_jaws_rs1_139_joint: type revolute, parent standard_jaws_base_link, child standard_jaws_rs1_139_link, origin xyz=0 -0.0155 0.0069 rpy=0 0 0, axis 1 0 0, limit lower=0 upper=0.5 effort=10 velocity=10, mimic joint=standard_jaws_rs1_130_joint multiplier=1 offset=0
- added joint tcp_joint: type fixed, parent standard_jaws_base_link, child tcp, origin xyz=0 0 0.09 rpy=0 0 0
- joint joint_1: limit lower=-3.072 upper=3.072 effort=9.0 velocity=0.5 -> lower=0 upper=5.725 effort=9.0 velocity=0.785
- joint joint_2: limit lower=-1.745 upper=1.745 effort=9.0 velocity=0.5 -> lower=-1.745 upper=1.745 effort=9.0 velocity=0.698
- joint joint_3: limit lower=-1.614 upper=1.614 effort=9.0 velocity=0.5 -> lower=0 upper=3.228 effort=9.0 velocity=0.698
- joint joint_4: limit lower=-0.785 upper=0.785 effort=9.0 velocity=0.5 -> lower=0 upper=5.725 effort=9.0 velocity=1.047
- joint joint_5: limit lower=0.001 upper=0.013 effort=10 velocity=10 -> lower=0.00137 upper=0.0133 effort=10 velocity=0.003; parent rs1_124_link -> ee_base_link

Commit message: copy the content of test file and paste it into the original urdf file.

File: alpha_description/urdf/alpha_robot_for_pybullet.urdf (robot description, URDF)
Before this commit: robot alpha_robot, 13 links, 12 joints
Joints:
- joint joint_1: limit lower=-3.072 upper=3.072 effort=9.0 velocity=0.5 -> lower=0 upper=5.725 effort=9.0 velocity=0.785
- joint joint_2: limit lower=-1.745 upper=1.745 effort=9.0 velocity=0.5 -> lower=-1.745 upper=1.745 effort=9.0 velocity=0.698
- joint joint_3: limit lower=-0.262 upper=2.094 effort=9.0 velocity=0.5 -> lower=0 upper=3.228 effort=9.0 velocity=0.698
- joint joint_4: limit lower=-2.862 upper=2.862 effort=9.0 velocity=0.5 -> lower=0 upper=5.725 effort=9.0 velocity=1.047
- joint joint_5: limit lower=0.001 upper=0.013 effort=10 velocity=10 -> lower=0.00137 upper=0.0133 effort=10 velocity=0.003

Commit message: Update alpha_robot_for_pybullet.urdf

File: alpha_description/urdf/alpha_robot_for_pybullet.urdf (robot description, URDF)
Before this commit: robot alpha_robot, 13 links, 12 joints
Links:
- link base_link: geometry collision cylinder length=0.150 radius=0.03; visual mesh filename=meshes/RS1-1010.dae
- link m1_link: geometry collision cylinder length=0.1 radius=0.03; visual mesh filename=meshes/M1.dae
- link m2_1_1_link: geometry collision cylinder length=0.033 radius=0.03; visual mesh filename=meshes/M2-1-1.dae
- link m2_1_3_link: geometry collision cylinder length=0.033 radius=0.03; visual mesh filename=meshes/M2-1-3.dae
- link m2_link: geometry collision cylinder length=0.040 radius=0.03; collision cylinder length=0.040 radius=0.03
- link m3_inline_link: geometry collision cylinder length=0.150 radius=0.03; visual mesh filename=meshes/M3-INLINE.dae
Joints:
- joint joint_1: limit lower=-3.072 upper=3.072 effort=9.0 velocity=0.5 -> lower=0 upper=5.725 effort=9.0 velocity=0.785
- joint joint_2: limit lower=-1.745 upper=1.745 effort=9.0 velocity=0.5 -> lower=-1.745 upper=1.745 effort=9.0 velocity=0.698
- joint joint_3: limit lower=-1.614 upper=1.614 effort=9.0 velocity=0.5 -> lower=0 upper=3.228 effort=9.0 velocity=0.698
- joint joint_4: limit lower=-0.785 upper=0.785 effort=9.0 velocity=0.5 -> lower=0 upper=5.725 effort=9.0 velocity=1.047
- joint joint_5: limit lower=0.001 upper=0.013 effort=10 velocity=10 -> lower=0.00137 upper=0.0133 effort=10 velocity=0.003

Commit message: please run train_v7.py, add curriculum learning, crossQ, TQC, and domain randomization

File: alpha_description/urdf/alpha_robot_for_pybullet.urdf (robot description, URDF)
Before this commit: robot alpha_robot, 13 links, 12 joints
Links:
- link base_link: geometry collision cylinder length=0.150 radius=0.05; visual mesh filename=meshes/RS1-1010.dae
- link m2_1_1_link: geometry collision cylinder length=0.033 radius=0.05; visual mesh filename=meshes/M2-1-1.dae
- link m2_link: geometry collision cylinder length=0.040 radius=0.03; collision cylinder length=0.040 radius=0.05
- link m3_inline_link: geometry collision cylinder length=0.150 radius=0.05; visual mesh filename=meshes/M3-INLINE.dae
Joints:
- joint tcp_joint: origin xyz=0 0 0.09 rpy=0 0 0 -> xyz=0 0 0.04 rpy=0 0 0

Commit message: correct URDF file

File: alpha_description/urdf/alpha_robot_for_pybullet.urdf (robot description, URDF)
Before this commit: robot alpha_robot, 13 links, 12 joints
Joints:
- joint joint_2: limit lower=-1.745 upper=1.745 effort=9.0 velocity=0.698 -> lower=0 upper=3.0 effort=9.0 velocity=0.698
- joint tcp_joint: origin xyz=0 0 0.09 rpy=0 0 0 -> xyz=0 0 0.04 rpy=0 0 0

Commit message: play ground

File: alpha_description/urdf/alpha_robot_for_pybullet.urdf (robot description, URDF)
Before this commit: robot alpha_robot, 13 links, 12 joints
Links:
- link base_link: geometry collision cylinder length=0.150 radius=0.03; visual mesh filename=meshes/RS1-1010.dae
- link m2_1_1_link: geometry collision cylinder length=0.033 radius=0.03; visual mesh filename=meshes/M2-1-1.dae
- link m2_link: geometry collision cylinder length=0.040 radius=0.03; collision cylinder length=0.040 radius=0.03
- link m3_inline_link: geometry collision cylinder length=0.150 radius=0.03; visual mesh filename=meshes/M3-INLINE.dae
Joints:
- joint joint_2: limit lower=-1.745 upper=1.745 effort=9.0 velocity=0.698 -> lower=0 upper=3.0 effort=9.0 velocity=0.698

File: alpha_description/urdf/alpha_robot_for_pybullet_test.urdf (robot description, URDF)
Before this commit: robot alpha_robot, 13 links, 12 joints
Joints:
- joint joint_1: limit lower=0 upper=5.725 effort=9.0 velocity=0.785 -> lower=0 upper=5.725 effort=600.0 velocity=0.785
- joint joint_2: limit lower=-1.745 upper=1.745 effort=9.0 velocity=0.698 -> lower=0 upper=3.0 effort=600.0 velocity=0.698
- joint joint_3: limit lower=0 upper=3.228 effort=9.0 velocity=0.698 -> lower=0 upper=3.228 effort=600.0 velocity=0.698
- joint joint_4: limit lower=0 upper=5.725 effort=9.0 velocity=1.047 -> lower=0 upper=5.725 effort=600.0 velocity=1.047
- joint joint_5: limit lower=0.00137 upper=0.0133 effort=10 velocity=0.003 -> lower=0.00137 upper=0.0133 effort=600 velocity=0.003
- joint tcp_joint: origin xyz=0 0 0.09 rpy=0 0 0 -> xyz=0 0 0.04 rpy=0 0 0
